Commit message: Set the table's mass to 0.1

File: table_object/objects/large.urdf.xacro (robot description, xacro)
@@ -20,4 +20,5 @@
   <property name="table_y" value="-0.5" />
   <property name="table_z" value="0.0" />
+  <property name="table_mass" value="0.1" />
   <property name="table_top_thickness" value="0.05"/>
   <property name="M_PI" value="3.1415926535897931" />
@@ -25,5 +26,5 @@
   <link name="table_top_link">
     <inertial>
-      <mass value="1.0" />
+        <mass value="${table_mass}" />
       <origin xyz="${table_x} ${table_y} ${table_z+table_height-table_top_thickness/2}" />
       <inertia ixx="1" ixy="0"  ixz="0"
@@ -58,5 +59,5 @@
   <link name="leg1_link">
     <inertial>
-      <mass value="1.0" />
+    <mass value="${table_mass}" />
       <origin xyz="0 0 ${-table_height/2}" />
       <inertia ixx="0.1" ixy="0"  ixz="0"
@@ -92,5 +93,5 @@
   <link name="leg2_link">
     <inertial>
-      <mass value="1.0" />
+      <mass value="${table_mass}" />
       <origin xyz="0 0 ${-table_height/2}" />
       <inertia ixx="0.1" ixy="0"  ixz="0"
@@ -126,5 +127,5 @@
   <link name="leg3_link">
     <inertial>
-      <mass value="1.0" />
+      <mass value="${table_mass}" />
       <origin xyz="0 0 ${-table_height/2}" />
       <inertia ixx="0.1" ixy="0"  ixz="0"
@@ -160,5 +161,5 @@
   <link name="leg4_link">
     <inertial>
-      <mass value="1.0" />
+      <mass value="${table_mass}" />
       <origin xyz="0 0 ${-table_height/2}" />
       <inertia ixx="0.1" ixy="0"  ixz="0"
